File: KiCAD_files/Etch-a-Sketch.kicad_sch (KiCad schematic)
At the start: 54 parts, among them J1 Debug Connector, J2 Display / Mounting Socket, J3 Display Mounting Socket, J4 Molex 2171790001, P1 282837-2, U1 STM32L433CCTx, U2 W25Q64JV, U3 LIS2DH12TR, U4 MCP1700x-300xxTT, U5 PEC11R_4215F_S0024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

Commit message: Change Accelerometer IC
Parts:
- removed U3: LIS2DH12TR, LGA-12_STM, symbol LIS2DH12TR:LIS2DH12TR
- added U3: LIS3DHTR, LGA-16_3x3x1mm_STM, symbol 2026-05-08_15-18-50:LIS3DHTR
- C2: value 10uF -> 0.1uF
- C3: value 0.1uF -> 10uF
Connections:
- net +3V3: now also U3.1 (VDD_IO), U3.14 (VDD)
- net ACC_INT1: now also U1.25 (PB12), U3.11 (INT1); no longer U1.26 (PB13)
- net ACC_INT2: now also U1.26 (PB13), U3.9 (INT2); no longer U1.25 (PB12)
- net GND: now also U3.10 (RES), U3.12 (GND), U3.5 (GND)
- net SPI2_CS: now also U3.8 (CS)
- net SPI2_MICO: now also U3.7 (SDO/SA0)
- net SPI2_MOCI: now also U3.6 (SDA/SDI/SDO)
- net SPI2_SCK: now also U3.4 (SCL/SPC)
